Commit message: Modified code to function on Noetic (mostly)

File: src/allegro_hand_description/allegro_hand_description_right.urdf.xacro (robot description, xacro)
@@ -14,9 +14,4 @@
   <!-- ============================================================================= -->
   <!-- PALM -->
-  <!-- <link name="dummy_link"/>
-  <joint name="dummy_joint" type="fixed">
-    <parent link="dummy_link"/>
-    <child link="palm_link"/>
-  </joint> -->
   <link name="palm_link">
     <visual>

File: src/allegro_hand_description/allegro_hand_description_right.xacro (robot description, xacro)
@@ -75,4 +75,10 @@
     <!-- RIGHT HAND due to which finger is number 0 -->
     <!-- for LEFT HAND switch the sign of the **offset_origin_y** and **finger_angle_r** parameters-->
+    <!-- THREE FINGER MACRO -->
+    <xacro:macro name="finger"
+                 params="finger_num offset_origin_x offset_origin_y offset_origin_z finger_angle_r">
+    <!-- THUMB MACRO -->
+    <xacro:macro name="thumb_right"
+                 params="finger_num offset_origin_x offset_origin_y offset_origin_z finger_angle_r finger_angle_p finger_angle_y">
     <xacro:finger
             finger_num="0"
@@ -107,7 +113,4 @@
             />
     <!-- ============================================================================= -->
-    <!-- THUMB MACRO -->
-    <xacro:macro name="thumb_right"
-                 params="finger_num offset_origin_x offset_origin_y offset_origin_z finger_angle_r finger_angle_p finger_angle_y">
         <!-- [LINK 12] -->
         <link name="link_${finger_num*4+0}">
@@ -276,7 +279,4 @@
     </xacro:macro>
     <!-- END THUMB MACRO -->
-    <!-- THREE FINGER MACRO -->
-    <xacro:macro name="finger"
-                 params="finger_num offset_origin_x offset_origin_y offset_origin_z finger_angle_r">
         <!-- [LINK 0, 4, 8] -->
         <link name="link_${finger_num*4+0}">
